Commit message: improved hardware interface.

File: src/meca500_description/urdf/meca500.xacro (robot description, xacro)
@@ -1,3 +1,3 @@
-<robot name="meca500" xmlns:xacro="http://ros.org/wiki/xacro">
+<robot name="meca500_arm" xmlns:xacro="http://ros.org/wiki/xacro">
   <!-- Base link is the center of the robot's bottom plate -->
   <link name="meca_base_link">
@@ -5,5 +5,5 @@
       <origin xyz="0 0 0" rpy="0 0 0" />
       <geometry>
-        <mesh filename="package://meca500_description/meshes/meca_500_r3_base.dae" />
+        <mesh filename="package://meca500_description/meshes/visual/meca_500_r3_base.dae" />
       </geometry>
     </visual>
@@ -20,5 +20,5 @@
       <origin xyz="0 0 0" rpy="0 0 0" />
       <geometry>
-        <mesh filename="package://meca500_description/meshes/meca_500_r3_j1.dae" />
+        <mesh filename="package://meca500_description/meshes/visual/meca_500_r3_j1.dae" />
       </geometry>
     </visual>
@@ -42,5 +42,5 @@
       <origin xyz="0 0 0" rpy="0 0 0" />
       <geometry>
-        <mesh filename="package://meca500_description/meshes/meca_500_r3_j2.dae" />
+        <mesh filename="package://meca500_description/meshes/visual/meca_500_r3_j2.dae" />
       </geometry>
     </visual>
@@ -64,5 +64,5 @@
       <origin xyz="0 0 0" rpy="0 0 0" />
       <geometry>
-        <mesh filename="package://meca500_description/meshes/meca_500_r3_j3.dae" />
+        <mesh filename="package://meca500_description/meshes/visual/meca_500_r3_j3.dae" />
       </geometry>
     </visual>
@@ -86,5 +86,5 @@
       <origin xyz="0 0 0" rpy="0 0 0" />
       <geometry>
-        <mesh filename="package://meca500_description/meshes/meca_500_r3_j4.dae" />
+        <mesh filename="package://meca500_description/meshes/visual/meca_500_r3_j4.dae" />
       </geometry>
     </visual>
@@ -108,5 +108,5 @@
       <origin xyz="0 0 0" rpy="0 0 0" />
       <geometry>
-        <mesh filename="package://meca500_description/meshes/meca_500_r3_j5.dae" />
+        <mesh filename="package://meca500_description/meshes/visual/meca_500_r3_j5.dae" />
       </geometry>
     </visual>
@@ -130,5 +130,5 @@
       <origin xyz="0 0 0" rpy="0 0 0" />
       <geometry>
-        <mesh filename="package://meca500_description/meshes/meca_500_r3_j6.dae" />
+        <mesh filename="package://meca500_description/meshes/visual/meca_500_r3_j6.dae" />
       </geometry>
     </visual>

File: src/meca500_moveit/config/meca500.ros2_control.xacro (robot description, xacro)
@@ -10,25 +10,25 @@
             <param name="robot_port">10000</param>
         </hardware>
-        <joint name="joint_1">
+        <joint name="joint1">
             <command_interface name="position"/>
             <state_interface name="position"/>
         </joint>
-        <joint name="joint_2">
+        <joint name="joint2">
             <command_interface name="position"/>
             <state_interface name="position"/>
         </joint>
-        <joint name="joint_3">
+        <joint name="joint3">
             <command_interface name="position"/>
             <state_interface name="position"/>
         </joint>
-        <joint name="joint_4">
+        <joint name="joint4">
             <command_interface name="position"/>
             <state_interface name="position"/>
         </joint>
-        <joint name="joint_5">
+        <joint name="joint5">
             <command_interface name="position"/>
             <state_interface name="position"/>
         </joint>
-        <joint name="joint_6">
+        <joint name="joint6">
             <command_interface name="position"/>
             <state_interface name="position"/>

File: src/meca500_moveit/config/meca500.urdf.xacro (robot description, xacro)
@@ -1,5 +1,5 @@
 <?xml version="1.0"?>
 <!-- Author: Garrison Johnston 12/2025 -->
-<robot xmlns:xacro="http://www.ros.org/wiki/xacro" name="meca500">
+<robot xmlns:xacro="http://www.ros.org/wiki/xacro" name="meca500_arm">
     <xacro:arg name="initial_positions_file" default="initial_positions.yaml" />
     <!-- Import meca500 urdf file -->
@@ -7,4 +7,4 @@
     <!-- Import control_xacro -->
     <xacro:include filename="meca500.ros2_control.xacro" />
-    <xacro:meca500_ros2_control name="FakeSystem" initial_positions_file="$(arg initial_positions_file)"/>
+    <xacro:meca500_ros2_control name="$(arg hardware_type)" initial_positions_file="$(arg initial_positions_file)"/>
 </robot>
