Commit message: untested fix.

File: src/meca500_moveit/config/meca500.ros2_control.xacro (robot description, xacro)
@@ -2,11 +2,11 @@
 <!-- Author: Garrison Johnston 12/2025 -->
 <robot xmlns:xacro="http://www.ros.org/wiki/xacro">
-    <xacro:macro name="meca500_ros2_control" params="name initial_positions_file">
+    <xacro:macro name="meca500_ros2_control" params="name initial_positions_file hardware_plugin robot_ip robot_port">
         <xacro:property name="initial_positions" value="${load_yaml(initial_positions_file)['initial_positions']}"/>
         <ros2_control name="${name}" type="system">
         <hardware>
-            <plugin>meca500_hardware/Meca500Hardware</plugin>
-            <param name="robot_ip">192.168.0.100</param>
-            <param name="robot_port">10000</param>
+            <plugin>${hardware_plugin}</plugin>
+            <param name="robot_ip">${robot_ip}</param>
+            <param name="robot_port">${robot_port}</param>
         </hardware>
         <joint name="joint1">

File: src/meca500_moveit/config/meca500.urdf.xacro (robot description, xacro)
@@ -3,8 +3,17 @@
 <robot xmlns:xacro="http://www.ros.org/wiki/xacro" name="meca500_arm">
     <xacro:arg name="initial_positions_file" default="initial_positions.yaml" />
+    <xacro:arg name="hardware_plugin" default="mock_components/GenericSystem"/>
+    <xacro:arg name="robot_ip" default="192.168.0.100"/>
+    <xacro:arg name="robot_port" default="10000"/>
     <!-- Import meca500 urdf file -->
     <xacro:include filename="$(find meca500_description)/urdf/meca500.xacro" />
     <!-- Import control_xacro -->
     <xacro:include filename="meca500.ros2_control.xacro" />
-    <xacro:meca500_ros2_control name="$(arg hardware_type)" initial_positions_file="$(arg initial_positions_file)"/>
+    <xacro:meca500_ros2_control
+        name="$(arg hardware_type)"
+        hardware_plugin="$(arg hardware_plugin)"
+        robot_ip="$(arg robot_ip)"
+        robot_port="$(arg robot_port)"
+        initial_positions_file="$(arg initial_positions_file)"
+    />
 </robot>
